File: JTAGMux_1.0.sch (KiCad schematic (older format))
At the start: 13 parts, among them J1 Conn_02x10_Odd_Even, U1 SN74CBTLV16292DL

Commit message: complete version 1.0.0
Parts:
- removed D0, D1: LED0603, LED-0603, symbol SparkFun-LED:LED0603
- removed R0, R1: 68, 0603-RES, symbol SparkFun-Passives:RESISTOR0603-RES
- added D0, D1: LED, LED_SMD:LED_0603_1608Metric, symbol Device:LED
- added R0, R1: 68, Resistor_SMD:R_0603_1608Metric, symbol Device:R
- C0, C1: footprint 0603-CAP -> Capacitor_SMD:C_0603_1608Metric; symbol SparkFun-Capacitors:CAP0603-CAP -> Device:C
- J1, JTAG_IN0, JTAG_IN1, JTAG_OUT0: footprint (none) -> Connector_PinHeader_2.54mm:PinHeader_2x10_P2.54mm_Vertical
- PMOD_JA1, PMOD_JB1: footprint (none) -> Connector_PinHeader_2.54mm:PinHeader_2x06_P2.54mm_Horizontal
- U1: footprint Housings_SSOP:SSOP-56_7.5x18.5mm_Pitch0.635mm -> Package_SO:SSOP-56_7.5x18.5mm_P0.635mm; symbol aurel_libs:SN74CBTLV16292DL -> JTAGMux_1.0-rescue:SN74CBTLV16292DL-aurel_libs
Connections:
- net DBACK_in0: now also PMOD_JA1.7 (Pin_7)
- net DBRQ_in0: now also PMOD_JA1.8 (Pin_8)
- net GND: now also R0.2, R1.2
- net at U1.29 (12B2): now also D1.2 (A)
- net at U1.30 (12B1): now also D0.2 (A)
- removed net DBGACK_in0: PMOD_JA1.7 (Pin_7), PMOD_JA1.8 (Pin_8)
- new net: D1.1 (K), R1.1
- new net: D0.1 (K), R0.1

Commit message: version 1.0.1
Parts:
- PMOD_JA1, PMOD_JB1: footprint Connector_PinHeader_2.54mm:PinHeader_2x06_P2.54mm_Horizontal -> pmod_foortprint:PinHeader_2x06_P2.54mm_Horizontal_pmod
