File: JTAGMux_1.0.kicad_sch (KiCad schematic)
At the start: 13 parts, among them J1 Conn_02x10_Odd_Even, U1 SN74CBTLV16292DL

Commit message: Moved SN74CBTLV16292 in local lib with proper naming
Parts:
- U1: footprint Package_SO:SSOP-56_7.5x18.5mm_P0.635mm -> Housings_SSOP:SSOP-56_7.5x18.5mm_Pitch0.635mm; symbol JTAGMux_1.0-rescue:SN74CBTLV16292DL-aurel_libs -> JTAGMux_1.0-cache:SN74CBTLV16292DL
Changed lines of the file:
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@@
 	)
 	(symbol
-		(lib_id "JTAGMux_1.0-rescue:SN74CBTLV16292DL-aurel_libs")
+		(lib_id "JTAGMux_1.0-cache:SN74CBTLV16292DL")
 		(at 58.674 48.514 0)
 		(unit 1)
@@
 			)
 		)
-		(property "Footprint" "Package_SO:SSOP-56_7.5x18.5mm_P0.635mm"
+		(property "Footprint" "Housings_SSOP:SSOP-56_7.5x18.5mm_Pitch0.635mm"
 			(at 86.614 42.418 0)
 			(effects
